Commit message: ODROID-XU4 update

File: rugby/modeldescription/urdf/sensors/rplidar_laser.urdf.xacro (robot description, xacro)
@@ -6,5 +6,5 @@
 			<child link="rugby_rplidar"></child>
 			<!--  rotate z axis 180 degree according to the placement on angelbot -->
-			<origin xyz="0.0376 0.00015 0.128" rpy="0 0 3.1415"></origin>
+			<origin xyz="0.06 0.00075 0.22" rpy="0 0 3.1415"></origin>
 		</joint>
 	  	<link name="rugby_rplidar">
